File: Columna.sch (KiCad schematic (older format))
At the start: 9 parts, among them P1 CONN_01X21, P4 CONN_01X03

Commit message: Borro archivos y reacomodo general
Se borran archivos innecesarios para manejar el proyecto y se reacomodan algunos archivos que pertenecen a las librerías creadas para este cartel
Parts:
- P4: footprint Connect:Wafer_Vertical10x5.8x7RM2.5-3 -> Poste:Poste_1x3
Changed lines of the file:
@@
 EESchema Schematic File Version 2
-LIBS:Columna5060-rescue
 LIBS:power
 LIBS:device
@@
 LIBS:contrib
 LIBS:valves
+LIBS:jumper3_no
 LIBS:led_5060
 LIBS:TLC5940NT
-LIBS:jumper3_no
-LIBS:Columna5060-cache
+LIBS:Columna-cache
 EELAYER 25 0
 EELAYER END
@@
 F 0 "P4" H 6600 5900 50  0000 C CNN
 F 1 "CONN_01X03" V 6700 5700 50  0000 C CNN
-F 2 "Connect:Wafer_Vertical10x5.8x7RM2.5-3" H 6600 5700 50  0001 C CNN
+F 2 "Poste:Poste_1x3" H 6600 5700 50  0001 C CNN
 F 3 "" H 6600 5700 50  0000 C CNN
 	1    6600 5700
